File: src/onboard/2020_2021 Onboard Circuits/Navigationmark1.1.brd (EAGLE design)
At the start: 72.1 x 68.6 mm, 44 parts, among them IC1 A5975D, IC2 A5975D, IC3 CD74AC257M96

Commit message: Changed hole sizes for both board to 3mm for M3 screws and made boards slilghtly larger to have room around the holes without disrupting the wire traces. Updated photos of both boards.
Parts:
- removed U$2, U$3, U$4, U$5: (no value), holes:2,8
- added E$1, E$2, E$3, E$4: (no value), holes:3,0
- moved YELLOW 1.52 mm to (40.9, 63.8)
- moved BLUE 1.52 mm to (46.0, 63.8)
Routing:
- net GND: track 273.9 -> 273.3 mm
- net N$17: track 4.06 -> 4.70 mm
- net N$15: track 4.06 -> 4.70 mm
Other:
- board size 72.1 x 68.6 mm -> 76.6 x 68.6 mm
