File: src/onboard/2020_2021 Onboard Circuits/FinalSchematic1.2.brd (EAGLE design)
At the start: 137.6 x 80 mm, 85 parts, among them IC1 MIC2937A-5.0BT, IC3 A5975D

Commit message: Switched 6v LDO to MIC29310-5.0BT
Parts:
- IC1: value MIC2937A-5.0BT -> MIC29310-5.0BT
Changed lines of the file:
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@@
 <attribute name="VALUE" x="-34.798" y="-92.583" size="1.27" layer="27"/>
 </element>
-<element name="IC1" library="linear" library_urn="urn:adsk.eagle:library:262" package="TO220V" package3d_urn="urn:adsk.eagle:package:16417/2" value="MIC2937A-5.0BT" x="-29.972" y="-91.44" smashed="yes">
+<element name="IC1" library="linear" library_urn="urn:adsk.eagle:library:262" package="TO220V" package3d_urn="urn:adsk.eagle:package:16417/2" value="MIC29310-5.0BT" x="-29.972" y="-91.44" smashed="yes">
 <attribute name="NAME" x="-35.052" y="-97.4852" size="1.27" layer="25" ratio="10"/>
 <attribute name="POPULARITY" value="0" x="-29.972" y="-91.44" size="1.778" layer="27" display="off"/>
