File: src/ground-station/gnd-station_2023-2024_jlangl.sch (EAGLE design)
At the start: 9 parts, among them IC1 LM7805_TO220V, U1 ADAFRUIT_RFM95W_LORA_RADIO

Commit message: removed 3.3v regulator, spaced out wires
Parts:
- removed IC1: LM7805_TO220V, IC_Power-Management:LM7805_TO220V
Connections:
- removed net N$4: ARDUINO_NANO1.5V, IC1.VI
- net GND: no longer IC1.GND
- net LORA3.3V: now also ARDUINO_NANO1.5V; no longer IC1.VO
Changed lines of the file:
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@@
 <part name="H4" library="holes" library_urn="urn:adsk.eagle:library:237" deviceset="MOUNT-HOLE" device="2.8" package3d_urn="urn:adsk.eagle:package:14271/1"/>
 <part name="ARDUINO_NANO1" library="ArduinoNanoV30" deviceset="ARDUINO_NANO" device=""/>
-<part name="IC1" library="IC_Power-Management" deviceset="LM7805" device="_TO220V" package3d_urn="urn:adsk.eagle:package:16417/2"/>
 </parts>
 <sheets>
@@
 <attribute name="NAME" x="38.1" y="60.96" size="1.778" layer="95" rot="R270"/>
 <attribute name="VALUE" x="35.56" y="60.96" size="1.778" layer="96" rot="R270"/>
-</instance>
-<instance part="IC1" gate="G$1" x="93.98" y="10.16" smashed="yes">
-<attribute name="NAME" x="93.98" y="14.16" size="1.778" layer="95" align="center"/>
-<attribute name="VALUE" x="96.52" y="3.16" size="1.778" layer="96" align="center-left"/>
 </instance>
 </instances>
@@
 </segment>
 </net>
-<net name="N$4" class="0">
-<segment>
-<pinref part="ARDUINO_NANO1" gate="G$1" pin="5V"/>
-<wire x1="73.66" y1="25.4" x2="73.66" y2="10.16" width="0.1524" layer="91"/>
-<wire x1="73.66" y1="10.16" x2="83.82" y2="10.16" width="0.1524" layer="91"/>
-<pinref part="IC1" gate="G$1" pin="VI"/>
-</segment>
-</net>
 <net name="LORA3.3V" class="0">
 <segment>
-<pinref part="IC1" gate="G$1" pin="VO"/>
-<wire x1="104.14" y1="10.16" x2="111.76" y2="10.16" width="0.1524" layer="91"/>
-<label x="111.76" y="10.16" size="1.778" layer="95"/>
+<wire x1="73.66" y1="7.62" x2="81.28" y2="7.62" width="0.1524" layer="91"/>
+<label x="81.28" y="7.62" size="1.778" layer="95"/>
+<pinref part="ARDUINO_NANO1" gate="G$1" pin="5V"/>
+<wire x1="73.66" y1="25.4" x2="73.66" y2="7.62" width="0.1524" layer="91"/>
 </segment>
 <segment>
@@
 </segment>
 <segment>
-<pinref part="IC1" gate="G$1" pin="GND"/>
-<wire x1="93.98" y1="2.54" x2="93.98" y2="0" width="0.1524" layer="91"/>
-<label x="91.44" y="-2.54" size="1.778" layer="95"/>
-</segment>
-<segment>
