File: src/ground-station/gnd-station_jlangl_prod1.sch (EAGLE design)
At the start: 8 parts, among them U1 ADAFRUIT_RFM95W_LORA_RADIO

Commit message: first iteration of order board
Connections:
- new net CS: ARDUINO_NANO1.D8/CLK0, U1.CS
